Commit message: update cloud_robot

File: src/cloud_robot/urdf/ros2_control.xacro (robot description, xacro)
@@ -11,6 +11,6 @@
     <param name="left.max_accel">25.0</param>
     <param name="left.invert_direction">false</param>
-    <param name="left.front_enc_a">8</param>
-    <param name="left.front_enc_b">7</param>
+    <param name="left.front_enc_a">7</param>
+    <param name="left.front_enc_b">8</param>
     <param name="left.rear_enc_a">16</param>
     <param name="left.rear_enc_b">20</param>
@@ -66,4 +66,5 @@
     <param name="zero_offset_rad">2.35</param>
     <param name="invert">true</param>
+    <param name="max_velocity">2.0</param>
   </joint>
   <joint name="Revolucion_6">  <!--  right front flipper -->
@@ -77,4 +78,5 @@
     <param name="zero_offset_rad">2.35</param>
     <param name="invert">false</param>
+    <param name="max_velocity">2.0</param>
   </joint>
   <joint name="Revolucion_7">  <!--  right rear flipper -->
@@ -88,4 +90,5 @@
     <param name="zero_offset_rad">2.35</param>
     <param name="invert">true</param>
+    <param name="max_velocity">2.0</param>
   </joint>
   <joint name="Revolucion_8">  <!--  left rear flipper -->
@@ -99,4 +102,5 @@
     <param name="zero_offset_rad">2.35</param>
     <param name="invert">false</param>
+    <param name="max_velocity">2.0</param>
   </joint>
   <!-- ARM -->
@@ -111,4 +115,5 @@
     <param name="zero_offset_rad">2.35</param>
     <param name="invert">false</param>
+    <param name="max_velocity">0.8</param>
   </joint>
   <joint name="Revolucion_10"> <!--  joint 1 to joint bridge 1 -->
@@ -122,4 +127,5 @@
     <param name="zero_offset_rad">0</param>
     <param name="invert">false</param>
+    <param name="max_velocity">0.8</param>
   </joint>
   <joint name="Revolucion_11"> <!--  joint 1 to joint bridge 2 -->
@@ -133,4 +139,5 @@
     <param name="zero_offset_rad">0</param>
     <param name="invert">false</param>
+    <param name="max_velocity">0.8</param>
   </joint>
   <joint name="Revolucion_12">  <!--  joint bridge 2 to joint 2-->
@@ -144,6 +151,19 @@
     <param name="zero_offset_rad">0</param>
     <param name="invert">false</param>
+    <param name="max_velocity">0.8</param>
   </joint>
   <joint name="Revolucion_13"> <!--  joint 2 to  joint 3-->
+    <command_interface name="position"/>
+    <state_interface name="position"/>
+    <param name="channel">7</param>
+    <param name="rad_min">-2.35</param>
+    <param name="rad_max">2.35</param>
+    <param name="us_min">500</param>
+    <param name="us_max">2500</param>
+    <param name="zero_offset_rad">2.35</param>
+    <param name="invert">false</param>
+    <param name="max_velocity">0.8</param>
+  </joint>
+  <joint name="Revolucion_14"> <!--  joint 3 to  joint 4-->
     <command_interface name="position"/>
     <state_interface name="position"/>
@@ -155,6 +175,7 @@
     <param name="zero_offset_rad">2.35</param>
     <param name="invert">false</param>
+    <param name="max_velocity">0.8</param>
   </joint>
-  <joint name="Revolucion_14"> <!--  joint 3 to  joint 4-->
+  <joint name="Revolucion_15">  <!--  joint 4 to  joint 5-->
     <command_interface name="position"/>
     <state_interface name="position"/>
@@ -163,18 +184,8 @@
     <param name="rad_max">2.35</param>
     <param name="us_min">500</param>
-    <param name="us_max">2500</param>
+    <param name="us_max">2000</param>
     <param name="zero_offset_rad">2.35</param>
     <param name="invert">false</param>
-  </joint>
-  <joint name="Revolucion_15">  <!--  joint 4 to  joint 5-->
-    <command_interface name="position"/>
-    <state_interface name="position"/>
-    <param name="channel">10</param>
-    <param name="rad_min">-2.35</param>
-    <param name="rad_max">2.35</param>
-    <param name="us_min">500</param>
-    <param name="us_max">2500</param>
-    <param name="zero_offset_rad">2.35</param>
-    <param name="invert">false</param>
+    <param name="max_velocity">0.8</param>
   </joint>
 </ros2_control>
